Commit message: Update gz sim

File: robo_cart_description/urdf/gazebo_control.xacro (robot description, xacro)
@@ -10,5 +10,9 @@
             <wheel_separation>${base_width + wheel_length}</wheel_separation>
             <wheel_radius>${wheel_radius}</wheel_radius>
+            <frame_id>odom</frame_id>
+            <child_frame_id>base_footprint_link</child_frame_id>
         </plugin>
+        <plugin name="gz::sim::systems::JointStatePublisher"
+            filename="libgz-sim8-joint-state-publisher-system" />
     </gazebo>
 </robot>

File: robo_cart_description/urdf/robot.urdf.xacro (robot description, xacro)
@@ -1,28 +1,13 @@
 <?xml version="1.0"?>
 <robot xmlns:xacro="http://www.ros.org/wiki/xacro" name="robo_cart">
+    <xacro:arg name="use_ros2_control" default="false" />
     <!--<mesh filename="file://$(find robo_cart_description)/meshes/base.stl)" scale="1.0"/>-->
     <xacro:include filename="$(find robo_cart_description)/urdf/properties.xacro" />
     <xacro:include filename="$(find robo_cart_description)/urdf/base.xacro" />
-    <xacro:include filename="$(find robo_cart_description)/urdf/gazebo_control.xacro" />
-    <ros2_control name="ArduinoSystem" type="system">
-        <hardware>
-            <plugin>arduino_hardware/ArduinoHardwareInterface</plugin>
-        </hardware>
-        <joint name="base_front_left_wheel_joint">
-            <command_interface name="velocity" />
-            <state_interface name="position" />
-        </joint>
-        <joint name="base_front_right_wheel_joint">
-            <command_interface name="velocity" />
-            <state_interface name="position" />
-        </joint>
-        <joint name="base_rear_left_wheel_joint">
-            <command_interface name="velocity" />
-            <state_interface name="position" />
-        </joint>
-        <joint name="base_rear_right_wheel_joint">
-            <command_interface name="velocity" />
-            <state_interface name="position" />
-        </joint>
-    </ros2_control>
+    <xacro:if value="$(arg use_ros2_control)">
+        <xacro:include filename="$(find robo_cart_description)/urdf/ros2_control.xacro" />
+    </xacro:if>
+    <xacro:unless value="$(arg use_ros2_control)">
+        <xacro:include filename="$(find robo_cart_description)/urdf/gazebo_control.xacro" />
+    </xacro:unless>
 </robot>

File: robo_cart_description/urdf/ros2_control.xacro (robot description, xacro)
@@ -1,3 +1,24 @@
 <?xml version="1.0"?>
 <robot xmlns:xacro="http://www.ros.org/wiki/xacro">
+    <ros2_control name="ArduinoSystem" type="system">
+        <hardware>
+            <plugin>arduino_hardware/ArduinoHardwareInterface</plugin>
+        </hardware>
+        <joint name="base_front_left_wheel_joint">
+            <command_interface name="velocity" />
+            <state_interface name="position" />
+        </joint>
+        <joint name="base_front_right_wheel_joint">
+            <command_interface name="velocity" />
+            <state_interface name="position" />
+        </joint>
+        <joint name="base_rear_left_wheel_joint">
+            <command_interface name="velocity" />
+            <state_interface name="position" />
+        </joint>
+        <joint name="base_rear_right_wheel_joint">
+            <command_interface name="velocity" />
+            <state_interface name="position" />
+        </joint>
+    </ros2_control>
 </robot>
