Commit message: Update

File: robo_cart_description/urdf/robo_cart_ros2_control.urdf.xacro (robot description, xacro)
@@ -1,3 +1,3 @@
-<?xml version="1.0" ?>
+<?xml version="1.0"?>
 <robot xmlns:xacro="http://wiki.ros.org/xacro">
     <xacro:macro name="robo_cart_ros2_control" params="use_gazebo">
@@ -8,39 +8,57 @@
                     <plugin>gz_ros2_control/GazeboSimSystem</plugin>
                 </xacro:if>
+                <xacro:unless value="${use_gazebo}"><!-- if use_basebo is false -->
+                    <plugin>ros2_control_arduino_hw/RoboCartArduinoHW</plugin>
+                    <param name="front_left_joint_name">base_front_left_wheel_joint</param>
+                    <param name="front_right_joint_name">base_front_right_wheel_joint</param>
+                    <param name="back_left_joint_name">base_rear_left_wheel_join</param>
+                    <param name="back_right_joint_nam">base_rear_right_wheel_joint</param>
+                    <param name="loop_rate">100</param>
+                    <param name="device">/dev/arduino</param>
+                    <param name="baud_rate">115200</param>
+                    <param name="timeout_ms">1000</param>
+                    <param name="encoder_counts_per_revolution">20</param>
+                    <!-- Proportional Derivative Integral Output scaling -->
+                    <param name="pid_p">0</param>
+                    <param name="pid_d">0</param>
+                    <param name="pid_i">0</param>
+                    <param name="pid_o">0</param>
+                    <!-- all the other needed params -->
+                </xacro:unless>
             </hardware>
             <!-- we need another plugin for real hw if use_gazebo is false -->
             <joint name="base_front_left_wheel_joint">
-              <command_interface name="velocity">
-                  <param name="min">-50.0</param>
-                  <param name="max">50.0</param>
-              </command_interface>
-              <state_interface name="position"/>
-              <state_interface name="velocity"/>
-          </joint>
-          <joint name="base_front_right_wheel_joint">
-              <command_interface name="velocity">
-                  <param name="min">-50.0</param>
-                  <param name="max">50.0</param>
-              </command_interface>
-              <state_interface name="position"/>
-              <state_interface name="velocity"/>
-          </joint>
-          <joint name="base_rear_left_wheel_joint">
-              <command_interface name="velocity">
-                  <param name="min">-50.0</param>
-                  <param name="max">50.0</param>
-              </command_interface>
-              <state_interface name="position"/>
-              <state_interface name="velocity"/>
-          </joint>
-          <joint name="base_rear_right_wheel_joint">
-              <command_interface name="velocity">
-                  <param name="min">-50.0</param>
-                  <param name="max">50.0</param>
-              </command_interface>
-              <state_interface name="position"/>
-              <state_interface name="velocity"/>
-          </joint>
-      </ros2_control>
-  </xacro:macro>
+                <command_interface name="velocity">
+                    <param name="min">-50.0</param>
+                    <param name="max">50.0</param>
+                </command_interface>
+                <state_interface name="position" />
+                <state_interface name="velocity" />
+            </joint>
+            <joint name="base_front_right_wheel_joint">
+                <command_interface name="velocity">
+                    <param name="min">-50.0</param>
+                    <param name="max">50.0</param>
+                </command_interface>
+                <state_interface name="position" />
+                <state_interface name="velocity" />
+            </joint>
+            <joint name="base_rear_left_wheel_joint">
+                <command_interface name="velocity">
+                    <param name="min">-50.0</param>
+                    <param name="max">50.0</param>
+                </command_interface>
+                <state_interface name="position" />
+                <state_interface name="velocity" />
+            </joint>
+            <joint name="base_rear_right_wheel_joint">
+                <command_interface name="velocity">
+                    <param name="min">-50.0</param>
+                    <param name="max">50.0</param>
+                </command_interface>
+                <state_interface name="position" />
+                <state_interface name="velocity" />
+            </joint>
+        </ros2_control>
+    </xacro:macro>
 </robot>
