Commit message: Add camera

File: robo_cart_description/urdf/lidar.xacro (robot description, xacro)
@@ -1,9 +1,9 @@
 <?xml version="1.0"?>
 <robot xmlns:xacro="http://www.ros.org/wiki/xacro">
-    <xacro:macro name="load_lidar" params="base_length use_gazebo">
+    <xacro:macro name="load_lidar" params="base_length base_height use_gazebo">
         <joint name="base_laser_frame_joint" type="fixed">
             <parent link="base_link" />
             <child link="laser_frame" />
-            <origin xyz="${base_length / 4.0} 0 0.07" rpy="0 0 0" />
+            <origin xyz="${base_length / 4.0} 0 ${base_height + 0.055}" rpy="0 0 0" />
         </joint>
         <link name="laser_frame">
@@ -12,5 +12,5 @@
                 <geometry>
                     <mesh filename="file://$(find robo_cart_description)/meshes/X3_Lidar.stl"
-                        scale="0.008 0.008 0.008" />
+                        scale="0.001 0.001 0.001" />
                 </geometry>
                 <material name="black" />

File: robo_cart_description/urdf/robot.urdf.xacro (robot description, xacro)
@@ -1,11 +1,11 @@
 <?xml version="1.0"?>
 <robot xmlns:xacro="http://www.ros.org/wiki/xacro" name="robo_cart">
-    <xacro:arg name="use_gazebo" default="true" />
-    <xacro:arg name="wheel_radius" default="0.0325" />
-    <xacro:arg name="wheel_width" default="0.03040" />
+    <xacro:arg name="use_gazebo" default="false" />
+    <xacro:arg name="wheel_radius" default="0.03" />
+    <xacro:arg name="wheel_width" default="0.03" />
     <xacro:arg name="wheel_mass" default="0.047" />
     <xacro:arg name="base_length" default="0.256" />
     <xacro:arg name="base_width" default="0.1" />
-    <xacro:arg name="base_height" default="0.05" />
+    <xacro:arg name="base_height" default="0.063" />
     <xacro:arg name="base_mass" default="1.366" />
     <!--<mesh filename="file://$(find robo_cart_description)/meshes/base.stl)" scale="1.0"/>-->
@@ -17,5 +17,9 @@
         base_height="$(arg base_height)" base_mass="$(arg base_mass)" />
     <xacro:include filename="$(find robo_cart_description)/urdf/lidar.xacro" />
-    <xacro:load_lidar base_length="$(arg base_length)" use_gazebo="$(arg use_gazebo)" />
+    <xacro:load_lidar base_length="$(arg base_length)" base_height="$(arg base_height)"
+        use_gazebo="$(arg use_gazebo)" />
+    <xacro:include filename="$(find robo_cart_description)/urdf/camera.xacro" />
+    <xacro:load_camera base_length="$(arg base_length)" base_height="$(arg base_height)"
+        use_gazebo="$(arg use_gazebo)" />
     <xacro:include filename="$(find robo_cart_description)/urdf/velocity_control_plugin.xacro" />
     <xacro:load_velocity_control_plugin use_gazebo="$(arg use_gazebo)" />
