Commit message: Update docs

File: robo_cart_description/urdf/camera.xacro (robot description, xacro)
@@ -5,5 +5,5 @@
             <parent link="base_link" />
             <child link="camera_link" />
-            <origin xyz="${base_length / 2.0 + 0.009} 0 ${base_height + 0.02}" rpy="0 0 0" />
+            <origin xyz="${base_length / 2.0 + 0.009} 0 ${base_height + 0.02}" rpy="0 0.18 0" />
         </joint>
         <link name="camera_link">
