Commit message: Update

File: robo_cart_description/urdf/base.xacro (robot description, xacro)
@@ -28,8 +28,26 @@
         </link>
     </xacro:macro>
-    <link name="base_footprint_link" /><!-- the world link -->
+    <link name="odom"><!-- odom frame for Gazebo -->
+        <inertial>
+            <origin xyz="0.0 0.0 0.0" rpy="0.0 0.0 0.0" />
+            <mass value="0.001" />
+            <inertia ixx="0.001" ixy="0.0" ixz="0.0" iyy="0.001" iyz="0.0" izz="0.001" />
+        </inertial>
+    </link>
+    <joint name="odom_base_footprint_joint" type="fixed">
+        <parent link="odom" />
+        <child link="base_footprint_link" />
+        <origin xyz="0.0 0.0 0.0" rpy="0.0 0.0 0.0" />
+    </joint>
+    <link name="base_footprint_link"><!-- simplifies nav calcultions from 3d to 2d -->
+        <inertial>
+            <origin xyz="0.0 0.0 0.0" rpy="0.0 0.0 0.0" />
+            <mass value="0.001" />
+            <inertia ixx="0.001" ixy="0.0" ixz="0.0" iyy="0.001" iyz="0.0" izz="0.001" />
+        </inertial>
+    </link>
     <joint name="base_footprint_base_joint" type="fixed">
-        <parent link="base_footprint_link" /><!-- sets the relationship to the world link -->
-        <child link="base_link" /><!-- it'll be an error if relationship is not specified -->
+        <parent link="base_footprint_link" />
+        <child link="base_link" />
         <origin xyz="0.0 0.0 ${wheel_radius}" />
     </joint>

File: robo_cart_description/urdf/gazebo_control.xacro (robot description, xacro)
@@ -10,4 +10,5 @@
             <wheel_separation>${base_width + wheel_length}</wheel_separation>
             <wheel_radius>${wheel_radius}</wheel_radius>
+            <odom_topic>/odom</odom_topic>
             <frame_id>odom</frame_id>
             <child_frame_id>base_footprint_link</child_frame_id>

Commit message: Update

File: robo_cart_description/urdf/base.xacro (robot description, xacro)
@@ -28,23 +28,5 @@
         </link>
     </xacro:macro>
-    <link name="odom"><!-- odom frame for Gazebo -->
-        <inertial>
-            <origin xyz="0.0 0.0 0.0" rpy="0.0 0.0 0.0" />
-            <mass value="0.001" />
-            <inertia ixx="0.001" ixy="0.0" ixz="0.0" iyy="0.001" iyz="0.0" izz="0.001" />
-        </inertial>
-    </link>
-    <joint name="odom_base_footprint_joint" type="fixed">
-        <parent link="odom" />
-        <child link="base_footprint_link" />
-        <origin xyz="0.0 0.0 0.0" rpy="0.0 0.0 0.0" />
-    </joint>
-    <link name="base_footprint_link"><!-- simplifies nav calcultions from 3d to 2d -->
-        <inertial>
-            <origin xyz="0.0 0.0 0.0" rpy="0.0 0.0 0.0" />
-            <mass value="0.001" />
-            <inertia ixx="0.001" ixy="0.0" ixz="0.0" iyy="0.001" iyz="0.0" izz="0.001" />
-        </inertial>
-    </link>
+    <link name="base_footprint_link" /><!-- simplifies nav calcultions from 3d to 2d -->
     <joint name="base_footprint_base_joint" type="fixed">
         <parent link="base_footprint_link" />

File: robo_cart_description/urdf/gazebo_control.xacro (robot description, xacro)
@@ -10,7 +10,11 @@
             <wheel_separation>${base_width + wheel_length}</wheel_separation>
             <wheel_radius>${wheel_radius}</wheel_radius>
-            <odom_topic>/odom</odom_topic>
             <frame_id>odom</frame_id>
             <child_frame_id>base_footprint_link</child_frame_id>
+        </plugin>
+        <plugin name="gz::sim::systems::OdometryPublisher"
+            filename="libgz-sim8-odometry-publisher-system">
+            <odom_frame>odom</odom_frame>
+            <robot_base_frame>base_footprint_link</robot_base_frame>
         </plugin>
         <plugin name="gz::sim::systems::JointStatePublisher"

Commit message: Update gz sim

File: robo_cart_description/urdf/base.xacro (robot description, xacro)
@@ -1,32 +1,11 @@
 <?xml version="1.0"?>
 <robot xmlns:xacro="http://www.ros.org/wiki/xacro">
+    <xacro:arg name="prefix" default="base" />
     <xacro:property name="base_length" value="0.256" />
     <xacro:property name="base_width" value="0.1" />
     <xacro:property name="base_height" value="0.05" />
-    <xacro:property name="wheel_radius" value="0.03" />
-    <xacro:property name="wheel_length" value="0.01" />
     <xacro:property name="base_mass" value="1.366" />
-    <xacro:property name="wheel_mass" value="0.047" />
-    <xacro:macro name="wheel_link" params="prefix">
-        <link name="${prefix}_wheel_link">
-            <visual>
-                <geometry>
-                    <cylinder radius="${wheel_radius}" length="${wheel_length}" />
-                </geometry>
-                <origin xyz="0.0 0.0 0.0" rpy="${pi / 2.0} 0.0 0.0" />
-                <material name="black" />
-            </visual>
-            <collision>
-                <geometry>
-                    <sphere radius="${wheel_radius}" />
-                </geometry>
-                <origin xyz="0.0 0.0 0.0" rpy="0.0 0.0 0.0" />
-            </collision>
-            <xacro:cylinder_inertia m="${wheel_mass}" r="${wheel_radius}" l="${wheel_length}"
-                o_xyz="0 0 0"
-                o_rpy="${pi / 2.0} 0 0" />
-        </link>
-    </xacro:macro>
-    <link name="base_footprint_link" /><!-- simplifies nav calcultions from 3d to 2d -->
+    <xacro:include filename="$(find robo_cart_description)/urdf/mecanum_wheel.xacro" />
+    <link name="base_footprint_link" />
     <joint name="base_footprint_base_joint" type="fixed">
         <parent link="base_footprint_link" />
@@ -39,9 +18,6 @@
                 <box size="${base_length} ${base_width} ${base_height}" />
             </geometry>
-            <origin xyz="0.0 0.0 ${base_height / 2.0}" rpy="0.0 0.0 0.0" /><!-- add a link but not
-            modify the origin -->
-            <material name="white" /><!-- make sure to place inside the <visual> tag -->
-            <!-- <geometry>, <origin> and <material> tags should be direct children -->
-            <!-- of the <visual> tag -->
+            <origin xyz="0.0 0.0 ${base_height / 2.0}" rpy="0.0 0.0 0.0" />
+            <material name="white" />
         </visual>
         <collision>
@@ -54,35 +30,7 @@
             z="${base_height}" o_xyz="0 0 ${base_height / 2.0}" o_rpy="0 0 0" />
     </link>
-    <xacro:wheel_link prefix="front_right" />
-    <joint name="base_front_right_wheel_joint" type="continuous">
-        <parent link="base_link" />
-        <child link="front_right_wheel_link" />
-        <origin xyz="${base_length / 4.0} ${-(base_width + wheel_length) / 2.0} 0.0"
-            rpy="0.0 0.0 0.0" />
-        <axis xyz="0.0 1.0 0.0" /><!-- rotation axis y -->
-    </joint>
-    <xacro:wheel_link prefix="front_left" />
-    <joint name="base_front_left_wheel_joint" type="continuous">
-        <parent link="base_link" />
-        <child link="front_left_wheel_link" />
-        <origin xyz="${base_length / 4.0} ${(base_width + wheel_length) / 2.0} 0.0"
-            rpy="0.0 0.0 0.0" />
-        <axis xyz="0.0 1.0 0.0" /><!-- rotation axis y -->
-    </joint>
-    <xacro:wheel_link prefix="rear_right" />
-    <joint name="base_rear_right_wheel_joint" type="continuous">
-        <parent link="base_link" />
-        <child link="rear_right_wheel_link" />
-        <origin xyz="${-base_length / 4.0} ${-(base_width + wheel_length) / 2.0} 0.0"
-            rpy="0.0 0.0 0.0" />
-        <axis xyz="0.0 1.0 0.0" /><!-- rotation axis y -->
-    </joint>
-    <xacro:wheel_link prefix="rear_left" />
-    <joint name="base_rear_left_wheel_joint" type="continuous">
-        <parent link="base_link" />
-        <child link="rear_left_wheel_link" />
-        <origin xyz="${-base_length / 4.0} ${(base_width + wheel_length) / 2.0} 0.0"
-            rpy="0.0 0.0 0.0" />
-        <axis xyz="0.0 1.0 0.0" /><!-- rotation axis y -->
-    </joint>
+    <xacro:mecanum_wheel prefix="$(arg prefix)" side="front_right" x_reflect="1" y_reflect="-1" />
+    <xacro:mecanum_wheel prefix="$(arg prefix)" side="front_left" x_reflect="1" y_reflect="1" />
+    <xacro:mecanum_wheel prefix="$(arg prefix)" side="rear_right" x_reflect="-1" y_reflect="-1" />
+    <xacro:mecanum_wheel prefix="$(arg prefix)" side="rear_left" x_reflect="-1" y_reflect="1" />
 </robot>

File: robo_cart_description/urdf/gazebo_control.xacro (robot description, xacro)
@@ -8,5 +8,5 @@
             <back_right_joint>base_rear_right_wheel_joint</back_right_joint>
             <wheelbase>${base_length / 2.0}</wheelbase>
-            <wheel_separation>${base_width + wheel_length}</wheel_separation>
+            <wheel_separation>${base_width + wheel_width}</wheel_separation>
             <wheel_radius>${wheel_radius}</wheel_radius>
             <odom_publish_frequency>10.0</odom_publish_frequency>

Commit message: Update urdf

File: robo_cart_description/urdf/base.xacro (robot description, xacro)
@@ -1,36 +1,46 @@
 <?xml version="1.0"?>
 <robot xmlns:xacro="http://www.ros.org/wiki/xacro">
-    <xacro:arg name="prefix" default="base" />
-    <xacro:property name="base_length" value="0.256" />
-    <xacro:property name="base_width" value="0.1" />
-    <xacro:property name="base_height" value="0.05" />
-    <xacro:property name="base_mass" value="1.366" />
-    <xacro:include filename="$(find robo_cart_description)/urdf/mecanum_wheel.xacro" />
-    <link name="base_footprint_link" />
-    <joint name="base_footprint_base_joint" type="fixed">
-        <parent link="base_footprint_link" />
-        <child link="base_link" />
-        <origin xyz="0.0 0.0 ${wheel_radius}" />
-    </joint>
-    <link name="base_link">
-        <visual>
-            <geometry>
-                <box size="${base_length} ${base_width} ${base_height}" />
-            </geometry>
-            <origin xyz="0.0 0.0 ${base_height / 2.0}" rpy="0.0 0.0 0.0" />
-            <material name="white" />
-        </visual>
-        <collision>
-            <geometry>
-                <box size="${base_length} ${base_width} ${base_height}" />
-            </geometry>
-            <origin xyz="0.0 0.0 ${base_height / 2.0}" rpy="0.0 0.0 0.0" />
-        </collision>
-        <xacro:box_inertia m="${base_mass}" x="${base_length}" y="${base_width}"
-            z="${base_height}" o_xyz="0 0 ${base_height / 2.0}" o_rpy="0 0 0" />
-    </link>
-    <xacro:mecanum_wheel prefix="$(arg prefix)" side="front_right" x_reflect="1" y_reflect="-1" />
-    <xacro:mecanum_wheel prefix="$(arg prefix)" side="front_left" x_reflect="1" y_reflect="1" />
-    <xacro:mecanum_wheel prefix="$(arg prefix)" side="rear_right" x_reflect="-1" y_reflect="-1" />
-    <xacro:mecanum_wheel prefix="$(arg prefix)" side="rear_left" x_reflect="-1" y_reflect="1" />
+    <xacro:macro name="load_base"
+        params="use_gazebo wheel_radius wheel_width wheel_mass base_length base_width base_height base_mass">
+        <xacro:arg name="prefix" default="base" />
+        <link name="base_footprint_link" />
+        <joint name="base_footprint_base_joint" type="fixed">
+            <parent link="base_footprint_link" />
+            <child link="base_link" />
+            <origin xyz="0.0 0.0 ${wheel_radius}" />
+        </joint>
+        <link name="base_link">
+            <visual>
+                <geometry>
+                    <box size="${base_length} ${base_width} ${base_height}" />
+                </geometry>
+                <origin xyz="0.0 0.0 ${base_height / 2.0}" rpy="0.0 0.0 0.0" />
+                <material name="white" />
+            </visual>
+            <collision>
+                <geometry>
+                    <box size="${base_length} ${base_width} ${base_height}" />
+                </geometry>
+                <origin xyz="0.0 0.0 ${base_height / 2.0}" rpy="0.0 0.0 0.0" />
+            </collision>
+            <xacro:box_inertia m="${base_mass}" x="${base_length}" y="${base_width}"
+                z="${base_height}" o_xyz="0 0 ${base_height / 2.0}" o_rpy="0 0 0" />
+        </link>
+        <xacro:include filename="$(find robo_cart_description)/urdf/mecanum_wheel.xacro" />
+        <xacro:load_wheel wheel_mass="$(arg wheel_mass)" wheel_width="$(arg wheel_width)"
+            wheel_radius="$(arg wheel_radius)" use_gazebo="$(arg use_gazebo)" prefix="$(arg prefix)"
+            side="front_right" x_reflect="1" y_reflect="-1" />
+        <xacro:include filename="$(find robo_cart_description)/urdf/mecanum_wheel.xacro" />
+        <xacro:load_wheel wheel_mass="$(arg wheel_mass)" wheel_width="$(arg wheel_width)"
+            wheel_radius="$(arg wheel_radius)" use_gazebo="$(arg use_gazebo)" prefix="$(arg prefix)"
+            side="front_left" x_reflect="1" y_reflect="1" />
+        <xacro:include filename="$(find robo_cart_description)/urdf/mecanum_wheel.xacro" />
+        <xacro:load_wheel wheel_mass="$(arg wheel_mass)" wheel_width="$(arg wheel_width)"
+            wheel_radius="$(arg wheel_radius)" use_gazebo="$(arg use_gazebo)" prefix="$(arg prefix)"
+            side="rear_right" x_reflect="-1" y_reflect="-1" />
+        <xacro:include filename="$(find robo_cart_description)/urdf/mecanum_wheel.xacro" />
+        <xacro:load_wheel wheel_mass="$(arg wheel_mass)" wheel_width="$(arg wheel_width)"
+            wheel_radius="$(arg wheel_radius)" use_gazebo="$(arg use_gazebo)" prefix="$(arg prefix)"
+            side="rear_left" x_reflect="-1" y_reflect="1" />
+    </xacro:macro>
 </robot>

File: robo_cart_description/urdf/mecanum_wheel.xacro (robot description, xacro)
@@ -1,8 +1,6 @@
 <?xml version="1.0"?>
 <robot xmlns:xacro="http://www.ros.org/wiki/xacro">
-  <xacro:property name="wheel_radius" value="0.0325" />
-  <xacro:property name="wheel_width" value="0.03040" />
-  <xacro:property name="wheel_mass" value="0.047" />
-  <xacro:macro name="mecanum_wheel" params="prefix side x_reflect y_reflect">
+  <xacro:macro name="load_wheel"
+    params="wheel_mass wheel_radius wheel_width use_gazebo prefix side x_reflect y_reflect">
     <link name="${side}_wheel_link">
       <visual>
@@ -26,6 +24,5 @@
         <inertia
           ixx="${(wheel_mass/12.0) * (3*wheel_radius*wheel_radius + wheel_width*wheel_width)}"
-          ixy="0" ixz="0"
-          iyy="${(wheel_mass/2.0) * (wheel_radius*wheel_radius)}" iyz="0"
+          ixy="0" ixz="0" iyy="${(wheel_mass/2.0) * (wheel_radius*wheel_radius)}" iyz="0"
           izz="${(wheel_mass/12.0) * (3*wheel_radius*wheel_radius + wheel_width*wheel_width)}" />
       </inertial>
@@ -39,22 +36,24 @@
         rpy="0 0 0" />
     </joint>
-    <gazebo reference="${prefix}_${side}_wheel_link">
-      <surface>
-        <friction>
-          <ode>
-            <mu>1.0</mu>
-            <mu2>0.0</mu2>
-          </ode>
-        </friction>
-      </surface>
-      <visual>
-        <material>
-          <ambient>0.2 0.2 0.2 1.0</ambient>
-          <diffuse>0.2 0.2 0.2 1.0</diffuse>
-          <specular>0.2 0.2 0.2 1.0</specular>
-          <emissive>0.0 0.0 0.0 0.0</emissive>
-        </material>
-      </visual>
-    </gazebo>
+    <xacro:if value="${use_gazebo}">
+      <gazebo reference="${prefix}_${side}_wheel_link">
+        <surface>
+          <friction>
+            <ode>
+              <mu>1.0</mu>
+              <mu2>0.0</mu2>
+            </ode>
+          </friction>
+        </surface>
+        <visual>
+          <material>
+            <ambient>0.2 0.2 0.2 1.0</ambient>
+            <diffuse>0.2 0.2 0.2 1.0</diffuse>
+            <specular>0.2 0.2 0.2 1.0</specular>
+            <emissive>0.0 0.0 0.0 0.0</emissive>
+          </material>
+        </visual>
+      </gazebo>
+    </xacro:if>
   </xacro:macro>
 </robot>

File: robo_cart_description/urdf/robo_cart_ros2_control.xacro (robot description, xacro)
@@ -1,12 +1,11 @@
 <?xml version="1.0"?>
 <robot xmlns:xacro="http://wiki.ros.org/xacro">
-    <xacro:macro name="robo_cart_ros2_control" params="use_gazebo">
+    <xacro:macro name="load_robo_cart_ros2_control" params="use_gazebo">
         <ros2_control name="RoboCart" type="system">
             <hardware>
-                <xacro:if value="${use_gazebo}">
-                    <!-- we gonna be using Gazebo plugin if use_gazebo is true -->
+                <xacro:if value="${use_gazebo}"><!-- true if use_gazebo is true-->
                     <plugin>gz_ros2_control/GazeboSimSystem</plugin>
                 </xacro:if>
-                <xacro:unless value="${use_gazebo}"><!-- if use_basebo is false -->
+                <xacro:unless value="${use_gazebo}"><!-- true if use_gazebo is false -->
                     <plugin>ros2_control_arduino_hw/RoboCartArduinoHW</plugin>
                     <param name="front_left_joint_name">base_front_left_wheel_joint</param>

File: robo_cart_description/urdf/robot.urdf.xacro (robot description, xacro)
@@ -1,26 +1,26 @@
 <?xml version="1.0"?>
 <robot xmlns:xacro="http://www.ros.org/wiki/xacro" name="robo_cart">
-    <xacro:arg name="robot_name" default="robo_cart" />
-    <xacro:arg name="use_ros2_control" default="false" />
-    <xacro:arg name="use_gazebo" default="true" />
+    <xacro:arg name="use_gazebo" default="false" />
+    <xacro:arg name="wheel_radius" default="0.0325" />
+    <xacro:arg name="wheel_width" default="0.03040" />
+    <xacro:arg name="wheel_mass" default="0.047" />
+    <xacro:arg name="base_length" default="0.256" />
+    <xacro:arg name="base_width" default="0.1" />
+    <xacro:arg name="base_height" default="0.05" />
+    <xacro:arg name="base_mass" default="1.366" />
     <!--<mesh filename="file://$(find robo_cart_description)/meshes/base.stl)" scale="1.0"/>-->
     <xacro:include filename="$(find robo_cart_description)/urdf/properties.xacro" />
     <xacro:include filename="$(find robo_cart_description)/urdf/base.xacro" />
-    <xacro:if value="$(arg use_ros2_control)"><!-- true if use_ros2_control is true -->
-     <xacro:unless value="$(arg use_gazebo)"><!-- true if use_gazebo is false -->
-        <xacro:include filename="$(find robo_cart_description)/urdf/ros2_control.xacro" />
-    </xacro:unless>
-    </xacro:if>
-    <xacro:if value="$(arg use_gazebo)"><!-- true if use_gazebo is true -->
-    <xacro:unless value="$(arg use_ros2_control)"> <!-- true if use_ros2_control is false -->
-        <xacro:include filename="$(find robo_cart_description)/urdf/gazebo_control.xacro" /><!-- load basic config -->
-    </xacro:unless>
-    </xacro:if>
-    <!-- //////////////////////////////////////////////////////////////////////////  -->
-    <xacro:include filename="$(find robo_cart_description)/urdf/velocity_control_plugin.urdf.xacro" />
+    <xacro:load_base use_gazebo="$(arg use_gazebo)" wheel_radius="$(arg wheel_radius)"
+        wheel_width="$(arg wheel_width)" wheel_mass="$(arg wheel_mass)"
+        base_length="$(arg base_length)" base_width="$(arg base_width)"
+        base_height="$(arg base_height)" base_mass="$(arg base_mass)" />
+    <xacro:include filename="$(find robo_cart_description)/urdf/velocity_control_plugin.xacro" />
     <xacro:load_velocity_control_plugin use_gazebo="$(arg use_gazebo)" />
-    <xacro:include filename="$(find robo_cart_description)/urdf/gazebo_sim_ros2_control.urdf.xacro" />
-    <xacro:load_gazebo_sim_ros2_control_plugin robot_name="$(arg robot_name)" use_gazebo="$(arg use_gazebo)" />
-    <xacro:include filename="$(find robo_cart_description)/urdf/robo_cart_ros2_control.urdf.xacro" />
-    <xacro:robo_cart_ros2_control use_gazebo="$(arg use_gazebo)" />
+    <xacro:include filename="$(find robo_cart_description)/urdf/gazebo_sim_ros2_control.xacro" />
+    <xacro:load_gazebo_sim_ros2_control_plugin use_gazebo="$(arg use_gazebo)"
+        base_length="$(arg base_length)" base_width="$(arg base_width)"
+        wheel_radius="$(arg wheel_radius)" wheel_width="$(arg wheel_width)" />
+    <xacro:include filename="$(find robo_cart_description)/urdf/robo_cart_ros2_control.xacro" />
+    <xacro:load_robo_cart_ros2_control use_gazebo="$(arg use_gazebo)" />
 </robot>

Commit message: Update

File: robo_cart_description/urdf/base.xacro (robot description, xacro)
@@ -13,7 +13,8 @@
             <visual>
                 <geometry>
-                    <box size="${base_length} ${base_width} ${base_height}" />
+                    <mesh filename="file://$(find robo_cart_description)/meshes/robo_cart.stl"
+                        scale="0.001 0.001 0.001" />
                 </geometry>
-                <origin xyz="0.0 0.0 ${base_height / 2.0}" rpy="0.0 0.0 0.0" />
+                <origin xyz="0.0 -0.1875 0.015" rpy="0.0 0.0 ${-M_PI/2.0}" />
                 <material name="white" />
             </visual>

File: robo_cart_description/urdf/camera.xacro (robot description, xacro)
@@ -5,5 +5,5 @@
             <parent link="base_link" />
             <child link="camera_link" />
-            <origin xyz="${base_length / 2.0 + 0.009} 0 ${base_height + 0.02}" rpy="0 0.18 0" />
+            <origin xyz="${base_length / 2.0 + 0.009} 0 ${base_height + 0.02 + 0.015}" rpy="0 0.18 0" />
         </joint>
         <link name="camera_link">

File: robo_cart_description/urdf/lidar.xacro (robot description, xacro)
@@ -9,5 +9,5 @@
         <link name="laser_frame">
             <visual>
-                <origin xyz="0.0 -0.004 0.0" rpy="0.0 0.0 ${-M_PI}" />
+                <origin xyz="0.0 -0.004 0.015" rpy="0.0 0.0 ${-M_PI}" />
                 <geometry>
                     <mesh filename="file://$(find robo_cart_description)/meshes/X3_Lidar.stl"
@@ -21,5 +21,5 @@
                 </geometry>
             </collision>
-            <xacro:cylinder_inertia m="0.020" r="0.032" l="0.018" o_xyz="0 0 0" o_rpy="0 0 0" />
+            <xacro:cylinder_inertia m="0.020" r="0.032" l="0.018" o_xyz="0 0 0.015" o_rpy="0 0 0" />
         </link>
         <xacro:if value="${use_gazebo}">

File: robo_cart_description/urdf/mecanum_wheel.xacro (robot description, xacro)
@@ -7,5 +7,6 @@
         <origin xyz="0 0 0" rpy="${pi/2} 0 0" />
         <geometry>
-          <mesh filename="file://$(find robo_cart_description)/meshes/${side}_wheel.STL" />
+          <mesh filename="file://$(find robo_cart_description)/meshes/${side}_wheel.STL"
+            scale="0.9 0.9 0.9" />
         </geometry>
         <material name="dark_gray">
@@ -33,5 +34,5 @@
       <child link="${side}_wheel_link" />
       <origin
-        xyz="${(x_reflect * base_length) / 4.0} ${(y_reflect * (base_width + wheel_width)) / 2.0} 0.0"
+        xyz="${(x_reflect * base_length) / 4.0 - (x_reflect * 0.0055)} ${(y_reflect * (base_width + wheel_width)) / 2.0} 0.0"
         rpy="0 0 0" />
     </joint>
